File: mcu.sch (KiCad schematic (older format))
At the start: 16 parts, among them U4 CP2104-F03-GM, U5 OSC, U6 STM32F030F4

Commit message: Finish layout and routing of initial PCB revision.
Parts:
- C22, C25, C26, C27, C28, C29: footprint (none) -> Capacitors_SMD:C_0402
- C23, C24: footprint (none) -> Capacitors_SMD:C_0603
- R23, R24, R25, R26, R27: footprint (none) -> Resistors_SMD:R_0402
- U4: footprint (none) -> Housings_DFN_QFN:QFN-24-1EP_4x4mm_Pitch0.5mm
- U5: footprint MODULE -> bce:SIOSC
- U6: footprint (none) -> Housings_SSOP:TSSOP-20_4.4x6.5mm_Pitch0.65mm
Changed lines of the file:
@@
 LIBS:bce
 LIBS:stm32
+LIBS:usbsupply-cache
 EELAYER 25 0
 EELAYER END
@@
 F 0 "U4" H 3550 2450 60  0000 L BNN
 F 1 "CP2104-F03-GM" H 3550 140 60  0000 L BNN
-F 2 "" H 3550 2450 60  0000 C CNN
+F 2 "Housings_DFN_QFN:QFN-24-1EP_4x4mm_Pitch0.5mm" H 3550 2450 60  0001 C CNN
 F 3 "" H 3550 2450 60  0000 C CNN
 	1    3550 2450
@@
 $EndComp
 $Comp
-L +5V #PWR41
+L +5V #PWR037
 U 1 1 569E6CCC
 P 3050 2400
-F 0 "#PWR41" H 3050 2250 50  0001 C CNN
+F 0 "#PWR037" H 3050 2250 50  0001 C CNN
 F 1 "+5V" H 3050 2540 50  0000 C CNN
 F 2 "" H 3050 2400 50  0000 C CNN
@@
 F 0 "C22" H 2475 2800 50  0000 L CNN
 F 1 "1u" H 2475 2600 50  0000 L CNN
-F 2 "" H 2488 2550 50  0000 C CNN
+F 2 "Capacitors_SMD:C_0402" H 2488 2550 50  0001 C CNN
 F 3 "" H 2450 2700 50  0000 C CNN
 	1    2450 2700
@@
 $EndComp
 $Comp
-L GND #PWR38
+L GND #PWR038
 U 1 1 569E6D2B
 P 2450 2850
-F 0 "#PWR38" H 2450 2600 50  0001 C CNN
+F 0 "#PWR038" H 2450 2600 50  0001 C CNN
 F 1 "GND" H 2450 2700 50  0000 C CNN
 F 2 "" H 2450 2850 50  0000 C CNN
@@
 F 0 "C23" H 2825 3450 50  0000 L CNN
 F 1 "4.7u" H 2825 3250 50  0000 L CNN
-F 2 "" H 2838 3200 50  0000 C CNN
+F 2 "Capacitors_SMD:C_0603" H 2838 3200 50  0001 C CNN
 F 3 "" H 2800 3350 50  0000 C CNN
 	1    2800 3350
@@
 $EndComp
 $Comp
-L GND #PWR39
+L GND #PWR039
 U 1 1 569E6DB5
 P 2800 3500
-F 0 "#PWR39" H 2800 3250 50  0001 C CNN
+F 0 "#PWR039" H 2800 3250 50  0001 C CNN
 F 1 "GND" H 2800 3350 50  0000 C CNN
 F 2 "" H 2800 3500 50  0000 C CNN
@@
 F 0 "R23" V 2330 2850 50  0000 C CNN
 F 1 "10k" V 2250 2850 50  0000 C CNN
-F 2 "" V 2180 2850 50  0000 C CNN
+F 2 "Resistors_SMD:R_0402" V 2180 2850 50  0001 C CNN
 F 3 "" H 2250 2850 50  0000 C CNN
 	1    2250 2850
@@
 $EndComp
 $Comp
-L +5V #PWR42
+L +5V #PWR040
 U 1 1 569E6EA3
 P 3100 4250
-F 0 "#PWR42" H 3100 4100 50  0001 C CNN
+F 0 "#PWR040" H 3100 4100 50  0001 C CNN
 F 1 "+5V" H 3100 4390 50  0000 C CNN
 F 2 "" H 3100 4250 50  0000 C CNN
@@
 NoConn ~ 3350 4100
 $Comp
-L GND #PWR44
+L GND #PWR041
 U 1 1 569E6ED3
 P 4850 4700
-F 0 "#PWR44" H 4850 4450 50  0001 C CNN
+F 0 "#PWR041" H 4850 4450 50  0001 C CNN
 F 1 "GND" H 4850 4550 50  0000 C CNN
 F 2 "" H 4850 4700 50  0000 C CNN
@@
 F 0 "C25" H 3175 4800 50  0000 L CNN
 F 1 "1u" H 3175 4600 50  0000 L CNN
-F 2 "" H 3188 4550 50  0000 C CNN
+F 2 "Capacitors_SMD:C_0402" H 3188 4550 50  0001 C CNN
 F 3 "" H 3150 4700 50  0000 C CNN
 	1    3150 4700
@@
 F 0 "C24" H 2925 4800 50  0000 L CNN
 F 1 "4.7u" H 2925 4600 50  0000 L CNN
-F 2 "" H 2938 4550 50  0000 C CNN
+F 2 "Capacitors_SMD:C_0603" H 2938 4550 50  0001 C CNN
 F 3 "" H 2900 4700 50  0000 C CNN
 	1    2900 4700
@@
 $EndComp
 $Comp
-L GND #PWR40
+L GND #PWR042
 U 1 1 569E70FE
 P 2900 4850
-F 0 "#PWR40" H 2900 4600 50  0001 C CNN
+F 0 "#PWR042" H 2900 4600 50  0001 C CNN
 F 1 "GND" H 2900 4700 50  0000 C CNN
 F 2 "" H 2900 4850 50  0000 C CNN
@@
 $EndComp
 $Comp
-L GND #PWR43
+L GND #PWR043
 U 1 1 569E7122
 P 3150 4850
-F 0 "#PWR43" H 3150 4600 50  0001 C CNN
+F 0 "#PWR043" H 3150 4600 50  0001 C CNN
 F 1 "GND" H 3150 4700 50  0000 C CNN
 F 2 "" H 3150 4850 50  0000 C CNN
@@
 VIO
 $Comp
-L +3.3V #PWR37
+L +3.3V #PWR044
 U 1 1 569E73C1
 P 2250 2700
-F 0 "#PWR37" H 2250 2550 50  0001 C CNN
+F 0 "#PWR044" H 2250 2550 50  0001 C CNN
 F 1 "+3.3V" H 2250 2840 50  0000 C CNN
 F 2 "" H 2250 2700 50  0000 C CNN
@@
 F 0 "U6" H 8050 3500 50  0000 C CNN
 F 1 "STM32F030F4" H 8050 3350 50  0000 C CNN
-F 2 "" H 8050 3450 60  0000 C CNN
+F 2 "Housings_SSOP:TSSOP-20_4.4x6.5mm_Pitch0.65mm" H 8050 3450 60  0001 C CNN
 F 3 "" H 8050 3450 60  0000 C CNN
 	1    8050 3450
@@
 F 0 "U5" H 8000 2300 50  0000 C CNN
 F 1 "OSC" H 8000 2500 50  0000 C CNN
-F 2 "MODULE" H 8000 2200 50  0001 C CNN
+F 2 "bce:SIOSC" H 8000 2200 50  0001 C CNN
 F 3 "DOCUMENTATION" H 8000 2600 50  0001 C CNN
 	1    8000 2400
@@
 F 0 "R24" V 7430 2200 50  0000 C CNN
 F 1 "10k" V 7350 2200 50  0000 C CNN
-F 2 "" V 7280 2200 50  0000 C CNN
+F 2 "Resistors_SMD:R_0402" V 7280 2200 50  0001 C CNN
 F 3 "" H 7350 2200 50  0000 C CNN
 	1    7350 2200
@@
 $EndComp
 $Comp
-L +3.3V #PWR46
+L +3.3V #PWR045
 U 1 1 569E917D
 P 7350 2050
-F 0 "#PWR46" H 7350 1900 50  0001 C CNN
+F 0 "#PWR045" H 7350 1900 50  0001 C CNN
 F 1 "+3.3V" H 7350 2190 50  0000 C CNN
 F 2 "" H 7350 2050 50  0000 C CNN
@@
 $EndComp
 $Comp
-L +3.3V #PWR51
+L +3.3V #PWR046
 U 1 1 569E91AA
 P 8550 2050
-F 0 "#PWR51" H 8550 1900 50  0001 C CNN
+F 0 "#PWR046" H 8550 1900 50  0001 C CNN
 F 1 "+3.3V" H 8550 2190 50  0000 C CNN
 F 2 "" H 8550 2050 50  0000 C CNN
@@
 F 0 "C29" H 9125 2300 50  0000 L CNN
 F 1 "10n" H 9125 2100 50  0000 L CNN
-F 2 "" H 9138 2050 50  0000 C CNN
+F 2 "Capacitors_SMD:C_0402" H 9138 2050 50  0001 C CNN
 F 3 "" H 9100 2200 50  0000 C CNN
 	1    9100 2200
@@
 $EndComp
 $Comp
-L GND #PWR52
+L GND #PWR047
 U 1 1 569E9259
 P 9100 2350
-F 0 "#PWR52" H 9100 2100 50  0001 C CNN
+F 0 "#PWR047" H 9100 2100 50  0001 C CNN
 F 1 "GND" H 9100 2200 50  0000 C CNN
 F 2 "" H 9100 2350 50  0000 C CNN
@@
 $EndComp
 $Comp
-L GND #PWR47
+L GND #PWR048
 U 1 1 569E92B9
 P 7400 2600
-F 0 "#PWR47" H 7400 2350 50  0001 C CNN
+F 0 "#PWR048" H 7400 2350 50  0001 C CNN
 F 1 "GND" H 7400 2450 50  0000 C CNN
 F 2 "" H 7400 2600 50  0000 C CNN
@@
 F 0 "R25" V 8230 1550 50  0000 C CNN
 F 1 "10k" V 8150 1550 50  0000 C CNN
-F 2 "" V 8080 1550 50  0000 C CNN
+F 2 "Resistors_SMD:R_0402" V 8080 1550 50  0001 C CNN
 F 3 "" H 8150 1550 50  0000 C CNN
 	1    8150 1550
@@
 $EndComp
 $Comp
-L GND #PWR49
+L GND #PWR049
 U 1 1 569E953A
 P 8150 1700
-F 0 "#PWR49" H 8150 1450 50  0001 C CNN
+F 0 "#PWR049" H 8150 1450 50  0001 C CNN
 F 1 "GND" H 8150 1550 50  0000 C CNN
 F 2 "" H 8150 1700 50  0000 C CNN
@@
 SCL
 $Comp
-L +3.3V #PWR53
+L +3.3V #PWR050
 U 1 1 569E9CE2
 P 9300 2900
-F 0 "#PWR53" H 9300 2750 50  0001 C CNN
+F 0 "#PWR050" H 9300 2750 50  0001 C CNN
 F 1 "+3.3V" H 9300 3040 50  0000 C CNN
 F 2 "" H 9300 2900 50  0000 C CNN
@@
 $EndComp
 $Comp
-L GND #PWR54
+L GND #PWR051
 U 1 1 569E9DAE
 P 9300 4000
-F 0 "#PWR54" H 9300 3750 50  0001 C CNN
+F 0 "#PWR051" H 9300 3750 50  0001 C CNN
 F 1 "GND" H 9300 3850 50  0000 C CNN
 F 2 "" H 9300 4000 50  0000 C CNN
@@
 $EndComp
 $Comp
-L +3.3V #PWR48
+L +3.3V #PWR052
 U 1 1 569E9E93
 P 7600 900
-F 0 "#PWR48" H 7600 750 50  0001 C CNN
+F 0 "#PWR052" H 7600 750 50  0001 C CNN
 F 1 "+3.3V" H 7600 1040 50  0000 C CNN
 F 2 "" H 7600 900 50  0000 C CNN
@@
 F 0 "C26" H 7825 1150 50  0000 L CNN
 F 1 "100n" H 7825 950 50  0000 L CNN
-F 2 "" H 7838 900 50  0000 C CNN
+F 2 "Capacitors_SMD:C_0402" H 7838 900 50  0001 C CNN
 F 3 "" H 7800 1050 50  0000 C CNN
 	1    7800 1050
@@
 F 0 "C27" H 8075 1150 50  0000 L CNN
 F 1 "100n" H 8075 950 50  0000 L CNN
-F 2 "" H 8088 900 50  0000 C CNN
+F 2 "Capacitors_SMD:C_0402" H 8088 900 50  0001 C CNN
 F 3 "" H 8050 1050 50  0000 C CNN
 	1    8050 1050
@@
 F 0 "C28" H 8325 1150 50  0000 L CNN
 F 1 "1u" H 8325 950 50  0000 L CNN
-F 2 "" H 8338 900 50  0000 C CNN
+F 2 "Capacitors_SMD:C_0402" H 8338 900 50  0001 C CNN
 F 3 "" H 8300 1050 50  0000 C CNN
 	1    8300 1050
@@
 $EndComp
 $Comp
-L GND #PWR50
+L GND #PWR053
 U 1 1 569EA23E
 P 8500 1200
-F 0 "#PWR50" H 8500 950 50  0001 C CNN
+F 0 "#PWR053" H 8500 950 50  0001 C CNN
 F 1 "GND" H 8500 1050 50  0000 C CNN
 F 2 "" H 8500 1200 50  0000 C CNN
@@
 F 0 "R26" V 9530 950 50  0000 C CNN
 F 1 "3.3k" V 9450 950 50  0000 C CNN
-F 2 "" V 9380 950 50  0000 C CNN
+F 2 "Resistors_SMD:R_0402" V 9380 950 50  0001 C CNN
 F 3 "" H 9450 950 50  0000 C CNN
 	1    9450 950
@@
 $EndComp
 $Comp
-L +3.3V #PWR55
+L +3.3V #PWR054
 U 1 1 569EA769
 P 9450 800
-F 0 "#PWR55" H 9450 650 50  0001 C CNN
+F 0 "#PWR054" H 9450 650 50  0001 C CNN
 F 1 "+3.3V" H 9450 940 50  0000 C CNN
 F 2 "" H 9450 800 50  0000 C CNN
@@
 F 0 "R27" V 10330 950 50  0000 C CNN
 F 1 "3.3k" V 10250 950 50  0000 C CNN
-F 2 "" V 10180 950 50  0000 C CNN
+F 2 "Resistors_SMD:R_0402" V 10180 950 50  0001 C CNN
 F 3 "" H 10250 950 50  0000 C CNN
 	1    10250 950
@@
 $EndComp
 $Comp
-L +3.3V #PWR56
+L +3.3V #PWR055
 U 1 1 569EA89C
 P 10250 800
-F 0 "#PWR56" H 10250 650 50  0001 C CNN
+F 0 "#PWR055" H 10250 650 50  0001 C CNN
 F 1 "+3.3V" H 10250 940 50  0000 C CNN
 F 2 "" H 10250 800 50  0000 C CNN
@@
 	10050 1100 10250 1100
 $Comp
-L +3.3V #PWR45
+L +3.3V #PWR056
 U 1 1 569EAA8C
 P 6750 2850
-F 0 "#PWR45" H 6750 2700 50  0001 C CNN
+F 0 "#PWR056" H 6750 2700 50  0001 C CNN
 F 1 "+3.3V" H 6750 2990 50  0000 C CNN
 F 2 "" H 6750 2850 50  0000 C CNN
